Commit message: chore: promote leap workspace to top-level repo root

File: ros2_ws/src/leap1/xuegecar_description/urdf/xuegecar.urdf (robot description, URDF)
Before this commit: robot xuegecar, 7 links, 6 joints
Links:
- added link camera_link; visual box size=0.04 0.03 0.03
- added link ground_camera_link; visual box size=0.03 0.03 0.03
Joints:
- added joint camera_joint: type fixed, parent base_link, child camera_link, origin xyz=0.08 0.0 0.12 rpy=0 0 0
- added joint ground_camera_joint: type fixed, parent base_link, child ground_camera_link, origin xyz=-0.02 0.0 0.14 rpy=0 0 3.14159
